Commit message: Simplified the urdf of oscar
It can actually move around now

File: oscar_description/urdf/oscar.urdf (robot description, URDF)
Before this commit: robot OSCAR, 1 links, 0 joints
Links:
- added link left-wheel, mass 1; collision cylinder length=0.5 radius=0.035; visual cylinder length=0.5 radius=0.035
- added link right-wheel, mass 1; collision cylinder length=0.5 radius=0.035; visual cylinder length=0.5 radius=0.035
- link base_link: geometry collision box size=0.4 0.5 0.9; visual box size=0.4 0.5 0.9
Joints:
- added joint left-wheel-joint: type continuous, parent base_link, child left-wheel, origin xyz=0.2 0 -0.45, axis 0 1 0
- added joint right-wheel-joint: type continuous, parent base_link, child right-wheel, origin xyz=-0.2 0 -0.45, axis 0 1 0

Commit message: Improved URDF file
The oscar URDF file now has movable wheels

File: oscar_description/urdf/oscar.urdf (robot description, URDF)
Before this commit: robot OSCAR, 3 links, 2 joints
Links:
- removed link left-wheel
- removed link right-wheel
- added link aandrijf_links, mass 1.9885095139484; collision mesh filename=package://oscar_description/meshes/aandrijf_links.STL; visual mesh filename=package://oscar_description/meshes/aandrijf_links.STL
- added link aandrijfwiel_rechts, mass 1.98850951394841; collision mesh filename=package://oscar_description/meshes/aandrijfwiel_rechts.STL; visual mesh filename=package://oscar_description/meshes/aandrijfwiel_rechts.STL
- added link passief_links, mass 0.0275781208850642; collision mesh filename=package://oscar_description/meshes/passief_links.STL; visual mesh filename=package://oscar_description/meshes/passief_links.STL
- added link passief_rechts, mass 0.0275781208850642; collision mesh filename=package://oscar_description/meshes/passief_rechts.STL; visual mesh filename=package://oscar_description/meshes/passief_rechts.STL
- added link passief_wiel_links, mass 0.2926460297435; collision mesh filename=package://oscar_description/meshes/passief_wiel_links.STL; visual mesh filename=package://oscar_description/meshes/passief_wiel_links.STL
- added link passief_wiel_rechts, mass 0.29264656535805; collision mesh filename=package://oscar_description/meshes/passief_wiel_rechts.STL; visual mesh filename=package://oscar_description/meshes/passief_wiel_rechts.STL
- link base_link: mass 81.4616237556886 -> 31.6409583053883; geometry collision mesh filename=package://oscar_description/meshes/base_link.STL; visual mesh filename=package://oscar_description/meshes/base_link.STL
Joints:
- removed joint left-wheel-joint
- removed joint right-wheel-joint
- added joint motoras_rechts: type fixed, parent base_link, child aandrijfwiel_rechts, origin xyz=-0.0610091422953399 0.469275677790673 0.130661401040105 rpy=1.43463153506437 0.00686067939224516 1.57079137192323, axis 0 0 0
- added joint motoraslinks: type fixed, parent base_link, child aandrijf_links, origin xyz=-0.0610119665057251 -0.100710907612253 0.134571957615908 rpy=0.856802140670808 0.00686067939224831 1.57079137192323, axis 0 0 0
- added joint passief_wiel_rechts: type fixed, parent passief_rechts, child passief_wiel_rechts, origin xyz=0.0515096362203565 0.00999999999999988 0.000499999999915179 rpy=2.9256005116916 1.57079630572147 -3.06618110194042, axis 0 0 0
- added joint wiel_links_passief: type fixed, parent passief_links, child passief_wiel_links, origin xyz=0.0515096362203469 0.00999999999999997 -0.000499999999997314 rpy=2.3869575088601 1.5707963267949 0, axis 0 0 0
- added joint yrotatie_links_passief: type fixed, parent base_link, child passief_links, origin xyz=0.373806955642397 0.000686479005100441 0.045773429249947 rpy=1.56392069147652 0.0231730912705171 -0.000729862123761098, axis 0 0 0
- added joint yrotatie_rechts_passief: type fixed, parent base_link, child passief_rechts, origin xyz=0.373819879962153 0.367171554283413 0.0432587956780883 rpy=1.56291079697297 0.0228492297244313 -0.0446138555479234, axis 0 0 0
