Commit message: Used xacro macros to better organize differnent version of oscar

File: oscar_description/urdf/oscar.urdf.xacro (robot description, xacro)
@@ -1,25 +1,9 @@
 <?xml version="1.0"?>
-<robot name="oscar" xmlns:xacro="http://ros.org/wiki/xacro">
-  <!-- General -->
+<robot name="oscar" xmlns:xacro="http://www.ros.org/wiki/xacro">
+  <xacro:macro name="oscar" params="">
   <xacro:include filename="$(find oscar_description)/urdf/body.urdf.xacro"/>
   <xacro:include filename="$(find dpr4_description)/urdf/dpr4_description.urdf.xacro"/>
   <xacro:dpr4 name="base_link"/>
-  <gazebo>
-  <plugin name="differential_drive_controller" filename="libgazebo_ros_diff_drive.so">
-    <alwaysOn>true</alwaysOn>
-    <updateRate>10</updateRate>
-    <leftJoint>front_wheel_left_joint</leftJoint>
-    <rightJoint>front_wheel_right_joint</rightJoint>
-    <wheelSeparation>0.5380</wheelSeparation>
-    <wheelDiameter>0.2410</wheelDiameter>
-    <torque>20</torque>
-    <commandTopic>cmd_vel</commandTopic>
-    <odometryTopic>odom</odometryTopic>
-    <odometryFrame>odom</odometryFrame>
-    <robotBaseFrame>base_link</robotBaseFrame>
-    <legacyMode>false</legacyMode>
-    <odometrySource>true</odometrySource>
-  </plugin>
-</gazebo>
+  <xacro:oscar_body name="body" />
   <joint name="body_to_base" type="fixed">
     <origin xyz="0 0 0" rpy="0 0 0" />
@@ -27,3 +11,4 @@
     <child link="body" />
   </joint>
+</xacro:macro>
 </robot>
