Commit message: Started setup of rtabmap

File: oscar_description/urdf/body.urdf.xacro (robot description, xacro)
@@ -1,5 +1,5 @@
 <?xml version="1.0" encoding="UTF-8"?>
-<robot name="body" xmlns:xacro="http://ros.org/wiki/xacro"
-  xmlns:sensor="http://playerstage.sourceforge.net/gazebo/xmlschema/#sensor">
+<robot name="body" xmlns:xacro="http://ros.org/wiki/xacro"  xmlns:sensor="http://playerstage.sourceforge.net/gazebo/xmlschema/#sensor">
+  <include filename="$(find oscar_description)/urdf/sensors/sonar.urdf.xacro" />
   <link name="body">
     <inertial>
@@ -28,127 +28,4 @@
   <xacro:property name="kinect_pitch" value="${0.5 * pi}" />
   <link name="kinect_link">
-    <!-- <pose>0 0 0.05 0 0 0</pose> -->
-    <inertial>
-      <mass value="0.1" />
-      <inertia ixx="0.000166667" ixy="0" ixz="0" iyy="0.000166667" iyz="0" izz="0.000166667" />
-    </inertial>
-    <collision>
-      <origin xyz="0 0 0" rpy="0 0 0" />
-      <!-- <origin xyz="0 -0.1 0.72" rpy="${kinect_roll} ${kinect_pitch} 0" /> -->
-      <geometry>
-        <box size="0.1 0.1 0.1"/>
-      </geometry>
-    </collision>
-    <visual>
-      <origin xyz="0 0 0" rpy="0 0 0" />
-      <!-- <origin xyz="0 -0.1 0.72" rpy="${kinect_roll} ${kinect_pitch} 0" /> -->
-      <geometry>
-        <box size="0.1 0.1 0.1"/>
-      </geometry>
-    </visual>
-  </link>
-  <joint name="kinect_joint" type="fixed">
-    <origin xyz="0 -1 1" rpy="0 0 ${-0.5*pi}" />
-    <!-- <origin xyz="0 -0.1 0.72" rpy="${kinect_roll} ${kinect_pitch} 0" /> -->
-    <parent link="body" />
-    <child link="kinect_link" />
-  </joint>
-  <!-- <gazebo reference="${link_name}">
-    <sensor name="camera" type="depth">
-      <camera name="kinect_camera">
-        <horizontal_fov>1.047</horizontal_fov>
-        <image>
-          <width>320</width>
-          <height>240</height>
-        </image>
-        <clip>
-          <near>0.1</near>
-          <far>100</far>
-        </clip>
-      </camera>
-      <always_on>1</always_on>
-      <update_rate>30</update_rate>
-      <visualize>true</visualize>
-      <plugin name="${link_name}_controller" filename="libgazebo_ros_openni_kinect.so">
-        <baseline>0.2</baseline>
-        <alwaysOn>true</alwaysOn>
-        <updateRate>1.0</updateRate>
-        <cameraName>${camera_name}_ir</cameraName>
-        <imageTopicName>/${camera_name}/rgb/image_raw</imageTopicName>
-        <cameraInfoTopicName>/${camera_name}/depth/camera_info</cameraInfoTopicName>
-        <depthImageTopicName>/${camera_name}/depth/image_raw</depthImageTopicName>
-        <depthImageInfoTopicName>/${camera_name}/depth/camera_info</depthImageInfoTopicName>
-        <pointCloudTopicName>/${camera_name}/depth/points</pointCloudTopicName>
-        <frameName>${frame_name}</frameName>
-        <pointCloudCutoff>0.5</pointCloudCutoff>
-        <distortionK1>0.00000001</distortionK1>
-        <distortionK2>0.00000001</distortionK2>
-        <distortionK3>0.00000001</distortionK3>
-        <distortionT1>0.00000001</distortionT1>
-        <distortionT2>0.00000001</distortionT2>
-        <CxPrime>0</CxPrime>
-        <Cx>0</Cx>
-        <Cy>0</Cy>
-        <focalLength>0</focalLength>
-        <hackBaseline>0</hackBaseline>
-      </plugin>s
-    </sensor>
-  </gazebo> -->
-  <xacro:property name="name" value="first" />
-  <xacro:property name="fov" value="${15/360 * 2 * pi}" />
-  <xacro:property name="update_rate" value="300" />
-  <xacro:property name="minRange" value="0.02" />
-  <xacro:property name="maxRange" value="4" />
-  <xacro:property name="ros_topic" value="/test" />
-  <link name="${name}_link">
-      <inertial>
-        <origin xyz="0 0 0" rpy="0 0 0" />
-        <mass value="0.001" />
-        <inertia ixx="0.0001" ixy="0" ixz="0" iyy="0.000001" iyz="0" izz="0.0001" />
-      </inertial>
-    </link>
-    <joint name="${name}_joint" type="fixed">
-      <origin xyz="0 -0.5 1"/>
-      <parent link="body"/>
-      <child link="${name}_link"/>
-</joint>
-<gazebo reference="${name}_link">
-  <sensor type="ray" name="${name}">
-    <pose>0 0 0 0 0 0</pose>
-    <update_rate>${update_rate}</update_rate>
-    <visualize>false</visualize>
-    <ray>
-      <scan>
-        <horizontal>
-          <samples>5</samples>
-          <resolution>1</resolution>
-          <min_angle>-${fov/2}</min_angle>
-          <max_angle>${fov/2}</max_angle>
-        </horizontal>
-        <vertical>
-          <samples>5</samples>
-          <resolution>1</resolution>
-          <min_angle>-${fov/2}</min_angle>
-          <max_angle>${fov/2}</max_angle>
-        </vertical>
-      </scan>
-      <range>
-        <min>${minRange}</min>
-        <max>${maxRange}</max>
-        <resolution>0.01</resolution>
-      </range>
-    </ray>
-    <plugin filename="libgazebo_ros_range.so" name="gazebo_ros_range">
-      <gaussianNoise>0.005</gaussianNoise>
-      <alwaysOn>true</alwaysOn>
-      <updateRate>${update_rate}</updateRate>
-      <topicName>${ros_topic}</topicName>
-      <frameName>${name}_link</frameName>
-      <fov>${fov}</fov>
-      <radiation>ultrasound</radiation>
-    </plugin>
-  </sensor>
-</gazebo>
-  <!-- <link name="sonar_${name}">
     <inertial>
       <mass value="0.1" />
@@ -168,81 +45,106 @@
     </visual>
   </link>
-  <joint name="sonar_${name}_joint" type="fixed">
-    <origin xyz="0 -0.5 0.5" rpy="0 0 ${0*pi}" />
+  <joint name="kinect_joint" type="fixed">
+    <origin xyz="0 -1 1" rpy="0 0 ${-0.5*pi}" />
     <parent link="body" />
-    <child link="sonar_${name}" />
+    <child link="kinect_link" />
   </joint>
-  <gazebo reference="$sonar_{name}">
-     <sensor type="ray" name="sonar">
-       <pose>0 0 0 0 0 0</pose>
-       <update_rate>${update_rate}</update_rate>
-       <visualize>false</visualize>
-       <ray>
-         <scan>
-           <horizontal>
-             <samples>5</samples>
-             <resolution>1</resolution>
-             <min_angle>-${fov/2}</min_angle>
-             <max_angle>${fov/2}</max_angle>
-           </horizontal>
-           <vertical>
-             <samples>5</samples>
-             <resolution>1</resolution>
-             <min_angle>-${fov/2}</min_angle>
-             <max_angle>${fov/2}</max_angle>
-           </vertical>
-         </scan>
-         <range>
-           <min>${minRange}</min>
-           <max>${maxRange}</max>
-           <resolution>0.01</resolution>
-         </range>
-       </ray>
-       <plugin filename="libgazebo_ros_range.so" name="gazebo_ros_range">
-         <gaussianNoise>0.005</gaussianNoise>
-         <alwaysOn>1</alwaysOn>
-         <updateRate>${update_rate}</updateRate>
-         <topicName>${ros_topic}</topicName>
-         <fov>${fov}</fov>
-         <radiation>ultrasound</radiation>
-       </plugin>
-     </sensor>
-</gazebo> -->
-  <!-- <gazebo>
-    <sensor type="ray" name="sonar_${name}">
-           <pose>0 0 0 0 0 0</pose>
-           <update_rate>20</update_rate>
-           <visualize>true</visualize>
-           <ray>
-               <scan>
-                   <horizontal>
-                       <samples>47</samples>
-                       <resolution>1</resolution>
-                       <min_angle>-0.068</min_angle>
-                       <max_angle>0.068</max_angle>
-                   </horizontal>
-                   <vertical>
-                       <samples>47</samples>
-                       <resolution>1</resolution>
-                       <min_angle>-0.068</min_angle>
-                       <max_angle>0.068</max_angle>
-                   </vertical>
-               </scan>
-               <range>
-                   <min>0</min>
-                   <max>6.45</max>
-                   <resolution>0.0254</resolution>
-               </range>
-           </ray>
-           <plugin name="sonar_${name}_plugin" filename="libgazebo_ros_range.so">
-               <gaussianNoise>0.05</gaussianNoise>
-               <alwaysOn>true</alwaysOn>
-               <updateRate>20</updateRate>
-               <topicName>sonar/${name}</topicName>
-               <frameName>sonar_${name}_link</frameName>
-               <minRange>0.02</minRange>
-               <maxRange>4</maxRange>
-           </plugin>
-       </sensor>
+  <gazebo reference="${link_name}">
+    <sensor name="camera" type="depth">
+      <camera name="kinect_camera">
+        <horizontal_fov>1.047</horizontal_fov>
+        <image>
+          <width>320</width>
+          <height>240</height>
+        </image>
+        <clip>
+          <near>0.1</near>
+          <far>100</far>
+        </clip>
+      </camera>
+      <always_on>1</always_on>
+      <update_rate>30</update_rate>
+      <visualize>true</visualize>
+      <plugin name="${link_name}_controller" filename="libgazebo_ros_depth_camera.so">
+        <baseline>0.2</baseline>
+        <alwaysOn>true</alwaysOn>
+        <updateRate>1.0</updateRate>
+        <cameraName>${camera_name}_ir</cameraName>
+        <imageTopicName>/${camera_name}/rgb/image_raw</imageTopicName>
+        <cameraInfoTopicName>/${camera_name}/rgb/camera_info</cameraInfoTopicName>
+        <!-- <depthImageTopicName>/depth/image</depthImageTopicName> -->
+        <depthImageTopicName>/${camera_name}/depth/image_raw</depthImageTopicName>
+        <depthImageInfoTopicName>/${camera_name}/depth/camera_info</depthImageInfoTopicName>
+        <pointCloudTopicName>/${camera_name}/depth/points</pointCloudTopicName>
+        <frameName>${frame_name}</frameName>
+        <pointCloudCutoff>0.5</pointCloudCutoff>
+        <distortionK1>0.00000001</distortionK1>
+        <distortionK2>0.00000001</distortionK2>
+        <distortionK3>0.00000001</distortionK3>
+        <distortionT1>0.00000001</distortionT1>
+        <distortionT2>0.00000001</distortionT2>
+        <CxPrime>0</CxPrime>
+        <Cx>0</Cx>
+        <Cy>0</Cy>
+        <focalLength>0</focalLength>
+        <hackBaseline>0</hackBaseline>
+        </plugin>
+      </sensor>
+      </gazebo>
+      <xacro:property name="name" value="first" />
+      <xacro:property name="fov" value="${15/360 * 2 * pi}" />
+      <xacro:property name="update_rate" value="30" />
+      <xacro:property name="minRange" value="0.02" />
+      <xacro:property name="maxRange" value="4" />
+      <xacro:property name="ros_topic" value="/test" />
+      <xacro:sonar name="sonar1" fov="${fov}" update_rate="${update_rate}" minRange="${minRange}" maxRange="${maxRange}" ros_topic="/sonar" parent="body" x="1" y="1" z="1" roll="0" pitch="0" yaw="0"/>
+      <!-- <link name="${name}_link">
+      <inertial>
+        <origin xyz="0 0 0" rpy="0 0 0" />
+        <mass value="0.001" />
+        <inertia ixx="0.0001" ixy="0" ixz="0" iyy="0.000001" iyz="0" izz="0.0001" />
+      </inertial>
+    </link>
+    <joint name="${name}_joint" type="fixed">
+      <origin xyz="0 -0.5 1"/>
+      <parent link="body"/>
+      <child link="${name}_link"/>
+    </joint>
+    <gazebo reference="${name}_link">
+      <sensor type="ray" name="${name}">
+        <pose>0 0 0 0 0 0</pose>
+        <update_rate>${update_rate}</update_rate>
+        <visualize>false</visualize>
+        <ray>
+          <scan>
+            <horizontal>
+              <samples>5</samples>
+              <resolution>1</resolution>
+              <min_angle>-${fov/2}</min_angle>
+              <max_angle>${fov/2}</max_angle>
+            </horizontal>
+            <vertical>
+              <samples>5</samples>
+              <resolution>1</resolution>
+              <min_angle>-${fov/2}</min_angle>
+              <max_angle>${fov/2}</max_angle>
+            </vertical>
+          </scan>
+          <range>
+            <min>${minRange}</min>
+            <max>${maxRange}</max>
+            <resolution>0.01</resolution>
+          </range>
+        </ray>
+        <plugin filename="libgazebo_ros_range.so" name="gazebo_ros_range">
+          <gaussianNoise>0.005</gaussianNoise>
+          <alwaysOn>true</alwaysOn>
+          <updateRate>${update_rate}</updateRate>
+          <topicName>${ros_topic}</topicName>
+          <frameName>${name}_link</frameName>
+          <fov>${fov}</fov>
+          <radiation>ultrasound</radiation>
+        </plugin>
+      </sensor>
     </gazebo> -->
-</robot>
+  </robot>

File: oscar_description/urdf/oscar.urdf.xacro (robot description, xacro)
@@ -4,8 +4,8 @@
   <xacro:include filename="$(find oscar_description)/urdf/body.urdf.xacro"/>
   <xacro:include filename="$(find dpr4_description)/urdf/dpr4_description.urdf.xacro"/>
-  <!-- <gazebo>
+  <gazebo>
   <plugin name="differential_drive_controller" filename="libgazebo_ros_diff_drive.so">
     <alwaysOn>true</alwaysOn>
-    <updateRate>100</updateRate>
+    <updateRate>10</updateRate>
     <leftJoint>front_wheel_left_joint</leftJoint>
     <rightJoint>front_wheel_right_joint</rightJoint>
@@ -18,6 +18,7 @@
     <robotBaseFrame>base_link</robotBaseFrame>
     <legacyMode>false</legacyMode>
+    <odometrySource>true</odometrySource>
   </plugin>
-</gazebo> -->
+</gazebo>
   <joint name="body_to_base" type="fixed">
     <origin xyz="0 0 0" rpy="0 0 0" />

Commit message: Moved sensors to seperate xacro urdf files

File: oscar_description/urdf/body.urdf.xacro (robot description, xacro)
@@ -1,150 +1,25 @@
 <?xml version="1.0" encoding="UTF-8"?>
 <robot name="body" xmlns:xacro="http://ros.org/wiki/xacro"  xmlns:sensor="http://playerstage.sourceforge.net/gazebo/xmlschema/#sensor">
-  <include filename="$(find oscar_description)/urdf/sensors/sonar.urdf.xacro" />
-  <link name="body">
-    <inertial>
-      <origin xyz="0 0.27093 0.68573" rpy="0 0 0" />
-      <mass value="9.21868409" />
-      <inertia ixx="0.6" ixy="0" ixz="0" iyy="0.6" iyz="0" izz="0.24" />
-    </inertial>
-    <visual>
-      <origin xyz="0 0 0" rpy="0 0 0" />
-      <geometry>
-        <mesh filename="package://oscar_description/meshes/body.STL" />
-      </geometry>
-    </visual>
-    <collision>
-      <origin xyz="0 0 0" rpy="0 0 0" />
-      <geometry>
-        <mesh filename="package://oscar_description/meshes/body.STL" />
-      </geometry>
-    </collision>
-  </link>
-  <xacro:property name="camera_name" value="kinect" />
-  <xacro:property name="frame_name" value="kinect_link" />
-  <xacro:property name="link_name" value="kinect_link" />
-  <xacro:property name="pi" value="3.1415926535897931" />
-  <xacro:property name="kinect_roll" value="${0.5 * pi}" />
-  <xacro:property name="kinect_pitch" value="${0.5 * pi}" />
-  <link name="kinect_link">
-    <inertial>
-      <mass value="0.1" />
-      <inertia ixx="0.000166667" ixy="0" ixz="0" iyy="0.000166667" iyz="0" izz="0.000166667" />
-    </inertial>
-    <collision>
-      <origin xyz="0 0 0" rpy="0 0 0" />
-      <geometry>
-        <box size="0.1 0.1 0.1"/>
-      </geometry>
-    </collision>
-    <visual>
-      <origin xyz="0 0 0" rpy="0 0 0" />
-      <geometry>
-        <box size="0.1 0.1 0.1"/>
-      </geometry>
-    </visual>
-  </link>
-  <joint name="kinect_joint" type="fixed">
-    <origin xyz="0 -1 1" rpy="0 0 ${-0.5*pi}" />
-    <parent link="body" />
-    <child link="kinect_link" />
-  </joint>
-  <gazebo reference="${link_name}">
-    <sensor name="camera" type="depth">
-      <camera name="kinect_camera">
-        <horizontal_fov>1.047</horizontal_fov>
-        <image>
-          <width>320</width>
-          <height>240</height>
-        </image>
-        <clip>
-          <near>0.1</near>
-          <far>100</far>
-        </clip>
-      </camera>
-      <always_on>1</always_on>
-      <update_rate>30</update_rate>
-      <visualize>true</visualize>
-      <plugin name="${link_name}_controller" filename="libgazebo_ros_depth_camera.so">
-        <baseline>0.2</baseline>
-        <alwaysOn>true</alwaysOn>
-        <updateRate>1.0</updateRate>
-        <cameraName>${camera_name}_ir</cameraName>
-        <imageTopicName>/${camera_name}/rgb/image_raw</imageTopicName>
-        <cameraInfoTopicName>/${camera_name}/rgb/camera_info</cameraInfoTopicName>
-        <!-- <depthImageTopicName>/depth/image</depthImageTopicName> -->
-        <depthImageTopicName>/${camera_name}/depth/image_raw</depthImageTopicName>
-        <depthImageInfoTopicName>/${camera_name}/depth/camera_info</depthImageInfoTopicName>
-        <pointCloudTopicName>/${camera_name}/depth/points</pointCloudTopicName>
-        <frameName>${frame_name}</frameName>
-        <pointCloudCutoff>0.5</pointCloudCutoff>
-        <distortionK1>0.00000001</distortionK1>
-        <distortionK2>0.00000001</distortionK2>
-        <distortionK3>0.00000001</distortionK3>
-        <distortionT1>0.00000001</distortionT1>
-        <distortionT2>0.00000001</distortionT2>
-        <CxPrime>0</CxPrime>
-        <Cx>0</Cx>
-        <Cy>0</Cy>
-        <focalLength>0</focalLength>
-        <hackBaseline>0</hackBaseline>
-        </plugin>
-      </sensor>
-      </gazebo>
-      <xacro:property name="name" value="first" />
-      <xacro:property name="fov" value="${15/360 * 2 * pi}" />
-      <xacro:property name="update_rate" value="30" />
-      <xacro:property name="minRange" value="0.02" />
-      <xacro:property name="maxRange" value="4" />
-      <xacro:property name="ros_topic" value="/test" />
-      <xacro:sonar name="sonar1" fov="${fov}" update_rate="${update_rate}" minRange="${minRange}" maxRange="${maxRange}" ros_topic="/sonar" parent="body" x="1" y="1" z="1" roll="0" pitch="0" yaw="0"/>
-      <!-- <link name="${name}_link">
+  <xacro:macro name="oscar_body" params="name">
+    <!-- <include filename="$(find oscar_description)/urdf/sensors/sonar.urdf.xacro" /> -->
+    <link name="${name}">
       <inertial>
+        <origin xyz="0 0.27093 0.68573" rpy="0 0 0" />
+        <mass value="9.21868409" />
+        <inertia ixx="0.6" ixy="0" ixz="0" iyy="0.6" iyz="0" izz="0.24" />
+      </inertial>
+      <visual>
         <origin xyz="0 0 0" rpy="0 0 0" />
-        <mass value="0.001" />
-        <inertia ixx="0.0001" ixy="0" ixz="0" iyy="0.000001" iyz="0" izz="0.0001" />
-      </inertial>
+        <geometry>
+          <mesh filename="package://oscar_description/meshes/body.STL" />
+        </geometry>
+      </visual>
+      <collision>
+        <origin xyz="0 0 0" rpy="0 0 0" />
+        <geometry>
+          <mesh filename="package://oscar_description/meshes/body.STL" />
+        </geometry>
+      </collision>
     </link>
-    <joint name="${name}_joint" type="fixed">
-      <origin xyz="0 -0.5 1"/>
-      <parent link="body"/>
-      <child link="${name}_link"/>
-    </joint>
-    <gazebo reference="${name}_link">
-      <sensor type="ray" name="${name}">
-        <pose>0 0 0 0 0 0</pose>
-        <update_rate>${update_rate}</update_rate>
-        <visualize>false</visualize>
-        <ray>
-          <scan>
-            <horizontal>
-              <samples>5</samples>
-              <resolution>1</resolution>
-              <min_angle>-${fov/2}</min_angle>
-              <max_angle>${fov/2}</max_angle>
-            </horizontal>
-            <vertical>
-              <samples>5</samples>
-              <resolution>1</resolution>
-              <min_angle>-${fov/2}</min_angle>
-              <max_angle>${fov/2}</max_angle>
-            </vertical>
-          </scan>
-          <range>
-            <min>${minRange}</min>
-            <max>${maxRange}</max>
-            <resolution>0.01</resolution>
-          </range>
-        </ray>
-        <plugin filename="libgazebo_ros_range.so" name="gazebo_ros_range">
-          <gaussianNoise>0.005</gaussianNoise>
-          <alwaysOn>true</alwaysOn>
-          <updateRate>${update_rate}</updateRate>
-          <topicName>${ros_topic}</topicName>
-          <frameName>${name}_link</frameName>
-          <fov>${fov}</fov>
-          <radiation>ultrasound</radiation>
-        </plugin>
-      </sensor>
-    </gazebo> -->
-  </robot>
+  </xacro:macro>
+</robot>
