Commit message: Rotated oscar so it points towards the positive x axis

File: oscar_description/robots/oscar_kinect.urdf.xacro (robot description, xacro)
@@ -4,9 +4,9 @@
 <xacro:include filename="$(find hector_sensors_description)/urdf/kinect_camera.urdf.xacro"/>
 <xacro:include filename="$(find hector_xacro_tools)/urdf/inertia_tensors.urdf.xacro"/>
-<xacro:kinect_camera_model name="habadabaduba_frame" parent="base_link" >
-  <origin xyz="0 0 0.73" rpy="0 0 ${1.5*M_PI}" />
+<xacro:kinect_camera_model name="kinect_model" parent="base_link" >
+  <origin xyz="0 0 0.73" rpy="0 0 ${0*M_PI}" />
 </xacro:kinect_camera_model>
-<xacro:kinect_camera name="habadabaduba" parent="base_link" >
-  <origin xyz="0 0 0.73" rpy="0 0 ${1.5*M_PI}" />
+<xacro:kinect_camera name="kinect" parent="base_link" >
+  <origin xyz="0 0 0.73" rpy="0 0 ${0*M_PI}" />
 </xacro:kinect_camera>
 <xacro:oscar />

File: oscar_description/urdf/body.urdf.xacro (robot description, xacro)
@@ -5,10 +5,10 @@
     <link name="${name}">
       <inertial>
-        <origin xyz="0 0.27093 0.68573" rpy="0 0 0" />
+        <origin xyz="-0.27093 0 0.68573" rpy="0 0 0" />
         <mass value="9.21868409" />
-        <inertia ixx="0.6" ixy="0" ixz="0" iyy="0.6" iyz="0" izz="0.24" />
+        <inertia iyy="0.6" ixy="0" ixz="0" ixx="0.6" iyz="0" izz="0.24" />
       </inertial>
       <visual>
-        <origin xyz="0 0 0" rpy="0 0 0" />
+        <origin xyz="0 0 0" rpy="0 0 1.57" />
         <geometry>
           <mesh filename="package://oscar_description/meshes/body.STL" />
@@ -16,5 +16,5 @@
       </visual>
       <collision>
-        <origin xyz="0 0 0" rpy="0 0 0" />
+        <origin xyz="0 0 0" rpy="0 0 1.57" />
         <geometry>
           <mesh filename="package://oscar_description/meshes/body.STL" />
